File: DogPathFinder/DogPathHelperCircuit.brd (EAGLE design)
At the start: 68.6 x 53.3 mm, 16 parts

Commit message: updated circuit file and image
Updated circuit file with image
Parts:
- added R6: (no value), AUTODESK_CIRCUITS_BREADBOARD:PHOTORESISTOR-2.54
- added R7: 10k‎Ω, AUTODESK_CIRCUITS_BREADBOARD:0207/10
Connections:
- removed net N$1 (its old number): PING1.2, PING2.2, PINGExternal sensor 3.2, PIR1.2, SERVO1.2, U1.5V
- removed net N$22 (its old number): U1.GND.
- new net N$24: R6.P$2, R7.1, U1.A0
- new net N$25: R7.2, U1.GND.
- new net N$26: PING1.2, PING2.2, PINGExternal sensor 3.2, PIR1.2, R6.P$1, SERVO1.2, U1.5V
